File: AD3D Cloud Connect Board.sch (KiCad schematic (older format))
At the start: 19 parts, among them J1 Conn_02x20_Odd_Even, J2 502585-04771, J3 Conn_01x03, J4 502585-04771, J5 Conn_01x03, J6 Conn_01x03, P1 NPTC202KFMS-RC, SW1 Reprint, SW2 Next, SW3 Unload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

Commit message: Revision 1. Fixed button orientations split out LEDs Changed to standard 0.1" headers
Parts:
- removed D1: APHB1608CGKSURKC, SamacSys_Parts:APHB1608CGKSURKC, symbol Device:LED_Dual_ACAC
- removed SW1: Reprint, AD3D custom footprints:PTS526-SK15-SMTR2-LFS, symbol AD3D~Cloud~Connect~Board:SPST_4pin
- removed SW2: Next, AD3D custom footprints:PTS526-SK15-SMTR2-LFS, symbol AD3D~Cloud~Connect~Board:SPST_4pin
- removed SW3: Unload, AD3D custom footprints:PTS526-SK15-SMTR2-LFS, symbol AD3D~Cloud~Connect~Board:SPST_4pin
- removed SW4: Load, AD3D custom footprints:PTS526-SK15-SMTR2-LFS, symbol AD3D~Cloud~Connect~Board:SPST_4pin
- removed SW5: Config, AD3D custom footprints:PTS526-SK15-SMTR2-LFS, symbol AD3D~Cloud~Connect~Board:SPST_4pin
- added D1: 150060RS75000, Diode_SMD:D_0603_1608Metric_Castellated, symbol Device:LED_Small
- added D2: 150060YS75000, Diode_SMD:D_0603_1608Metric_Castellated, symbol Device:LED_Small
- added D3: 150060VS75000‎, Diode_SMD:D_0603_1608Metric_Castellated, symbol Device:LED_Small
- added J7: Conn_01x02, Connector_PinHeader_2.54mm:PinHeader_1x02_P2.54mm_Vertical_SMD_Pin1Right, symbol Connector_Generic:Conn_01x02
- added R1: 82 OHM 5%, Resistor_SMD:R_0603_1608Metric, symbol Device:R_US
- added SW1: Config, AD3D custom footprints:SW_SPST_PTS647, symbol AD3D-Cloud-Connect-Board:SPST_4pin
- added SW2: Cancel/Offline, AD3D custom footprints:SW_SPST_PTS647, symbol AD3D-Cloud-Connect-Board:SPST_4pin
- added SW3: Next, AD3D custom footprints:SW_SPST_PTS647, symbol AD3D-Cloud-Connect-Board:SPST_4pin
- added SW4: Flmnt 1, AD3D custom footprints:SW_SPST_PTS647, symbol AD3D-Cloud-Connect-Board:SPST_4pin
- added SW5: Flmnt 2, AD3D custom footprints:SW_SPST_PTS647, symbol AD3D-Cloud-Connect-Board:SPST_4pin
- J1: footprint AD3D custom footprints:95157-440LF -> Connector_PinHeader_2.54mm:PinHeader_2x20_P2.54mm_Vertical_SMD
- J2, J4: value 502585-04771 -> Conn_01x04; footprint AD3D custom footprints:S4B-XH-SM4-TB -> Connector_PinHeader_2.54mm:PinHeader_1x04_P2.54mm_Vertical_SMD_Pin1Right; Note Black -> (none)
- J3, J5, J6: footprint AD3D custom footprints:S3B-XH-SM4-TB -> Connector_PinHeader_2.54mm:PinHeader_1x03_P2.54mm_Vertical_SMD_Pin1Right
- MK1, MK2, MK3, MK4: footprint MountingHole:MountingHole_2.7mm_M2.5 -> MountingHole:MountingHole_2.5mm
- P1: footprint AD3D custom footprints:NPTC202KFMS-RC -> Connector_PinSocket_2.54mm:PinSocket_2x20_P2.54mm_Vertical_SMD
Connections:
- wire segments 171 -> 188
Other:
- note added: "Power In"
- note added: "Yellow"
- note removed: "DNP = Do Not Populate"
- moved on the sheet: R7, R8
